Commit message: Initial commit

File: install/bumperbot_description/share/bumperbot_description/urdf/bumperbot.urdf.xacro (robot description, xacro)
@@ -69,3 +69,22 @@
         <origin rpy="0 0 0" xyz="-0.04755 0 -0.0275"/>
     </joint>
+<<<<<<< HEAD
+=======
+<<<<<<< HEAD
+=======
+    <link name="can_link">
+        <visual>
+            <origin rpy=" 1.57 0 0" xyz="-.0335 .0335 0"/>
+            <geometry>
+                <mesh filename="package://bumperbot_description/meshes/can.STL"/>
+            </geometry>
+        </visual>
+    </link>
+    <joint name="can_joint" type="fixed">
+        <parent link="base_link"/>
+        <child link="can_link"/>
+        <origin rpy=" 0 0 0" xyz="0 0 .078"/>
+    </joint>
+>>>>>>> 68b074e (Initial commit)
+>>>>>>> 81012a5 (Initial commit)
 </robot>

Commit message: added launch gazebo support

File: install/bumperbot_description/share/bumperbot_description/urdf/bumperbot.urdf.xacro (robot description, xacro)
@@ -1,6 +1,14 @@
 <?xml version="1.0"?>
 <robot xmlns:xacro="http://www.ros.org/wiki/xacro" name="bumperbot">
+    <xacro:include filename="$(find bumperbot_description)/urdf/bumperbot_gazebo.xacro"/>
     <link name="base_footprint"/>
     <link name="base_link">
+        <inertial>
+            <origin xyz="0 -0.014 0" rpy="0 0 0"/>
+            <mass value="0.0530086090966721"/>
+            <inertia ixx="1.88176298336665E-05" ixy="-4.8444933029987E-10" ixz="1.88163708851143E-08"
+                    iyy="3.11510738647764E-05" iyz="-6.93560663069607E-11"
+                    izz="1.8801969558182E-05"/>
+        </inertial>
         <visual>
             <origin rpy="0 0 0" xyz="0 0 0"/>
@@ -9,4 +17,10 @@
             </geometry>
         </visual>
+        <collision>
+            <origin rpy="0 0 0" xyz="0 0 0"/>
+            <geometry>
+                <mesh filename="package://bumperbot_description/meshes/base_link.STL"/>
+            </geometry>
+        </collision>
     </link>
     <joint name="base_joint" type="fixed">
@@ -16,4 +30,11 @@
     </joint>
     <link name="wheel_right_link">
+        <inertial>
+            <origin xyz="0 0.014 0" rpy="0 0 0"/>
+            <mass value="0.0530086043217644"/>
+            <inertia ixx="1.8792911368909E-05" ixy="3.31256392204584E-10" ixz="-1.14082001662767E-08"
+                    iyy="3.11510738759073E-05" iyz="-3.60499245082192E-10"
+                    izz="1.88266886146847E-05"/>
+</inertial>
         <visual>
             <origin rpy="1.57 0 0" xyz="0 0 0"/>
@@ -22,4 +43,10 @@
             </geometry>
         </visual>
+        <collision>
+            <origin xyz="0 -.015 0" rpy="1.57 0 0" />
+            <geometry>
+                <sphere radius="0.033"/>
+            </geometry>
+        </collision>
     </link>
     <joint name="wheel_right_joint" type="continuous">
@@ -30,4 +57,11 @@
     </joint>
     <link name="wheel_left_link">
+        <inertial>
+            <origin xyz="0 0.014 0" rpy="0 0 0"/>
+            <mass value="0.0530086043217644"/>
+            <inertia ixx="1.8792911368909E-05" ixy="3.31256392204584E-10" ixz="-1.14082001662767E-08"
+                    iyy="3.11510738759073E-05" iyz="-3.60499245082192E-10"
+                    izz="1.88266886146847E-05"/>
+        </inertial>
         <visual>
             <origin rpy="-1.57 0 0" xyz="0 0 0"/>
@@ -36,4 +70,10 @@
             </geometry>
         </visual>
+        <collision>
+            <origin xyz="0 .015 0" rpy="1.57 0 0" />
+            <geometry>
+                <sphere radius="0.033"/>
+            </geometry>
+        </collision>
     </link>
     <joint name="wheel_left_joint" type="continuous">
@@ -44,4 +84,11 @@
     </joint>
     <link name="caster_front_link">
+        <inertial>
+            <origin xyz="3.89968128948481E-07 2.40073004698083E-07 0.00219173397061506" rpy="0 0 0"/>
+            <mass value="1.44379265037903E-06"/>
+            <inertia ixx="7.23075276010246E-11" ixy="-6.10956883467859E-16" ixz="2.22849693525031E-15"
+                    iyy="3.8713793085917E-11" iyz="2.93909858781952E-15"
+                    izz="1.00967486676306E-10"/>
+        </inertial>
         <visual>
             <origin rpy="0 0 0" xyz="0 0 0"/>
@@ -50,4 +97,10 @@
             </geometry>
         </visual>
+        <collision>
+            <origin rpy="0 0 0" xyz="0 0 0"/>
+            <geometry>
+                <sphere radius="0.005"/>
+            </geometry>
+        </collision>
     </link>
     <joint name="caster_front_joint" type="fixed">
@@ -57,4 +110,11 @@
     </joint>
     <link name="caster_rear_link">
+        <inertial>
+            <origin xyz="3.8996812895542E-07 2.40073004698083E-07 0.00219173397061509" rpy="0 0 0"/>
+            <mass value="1.44379265037902E-06"/>
+            <inertia ixx="7.23075276010246E-11" ixy="-6.10956872363424E-16" ixz="2.22849693527207E-15"
+                    iyy="3.87137930859167E-11" iyz="2.939098587861E-15"
+                    izz="1.00967486676306E-10"/>
+        </inertial>
         <visual>
             <origin rpy="0 0 0" xyz="0 0 0"/>
@@ -63,4 +123,10 @@
             </geometry>
         </visual>
+        <collision>
+            <origin rpy="0 0 0" xyz="0 0 0"/>
+            <geometry>
+                <sphere radius="0.005"/>
+            </geometry>
+        </collision>
     </link>
     <joint name="caster_rear_joint" type="fixed">
@@ -69,8 +135,4 @@
         <origin rpy="0 0 0" xyz="-0.04755 0 -0.0275"/>
     </joint>
-<<<<<<< HEAD
-=======
-<<<<<<< HEAD
-=======
     <link name="can_link">
         <visual>
@@ -86,5 +148,3 @@
         <origin rpy=" 0 0 0" xyz="0 0 .078"/>
     </joint>
->>>>>>> 68b074e (Initial commit)
->>>>>>> 81012a5 (Initial commit)
 </robot>

File: src/bumperbot_description/urdf/bumperbot.urdf.xacro (robot description, xacro)
@@ -1,6 +1,14 @@
 <?xml version="1.0"?>
 <robot xmlns:xacro="http://www.ros.org/wiki/xacro" name="bumperbot">
+    <xacro:include filename="$(find bumperbot_description)/urdf/bumperbot_gazebo.xacro"/>
     <link name="base_footprint"/>
     <link name="base_link">
+        <inertial>
+            <origin xyz="0 -0.014 0" rpy="0 0 0"/>
+            <mass value="0.0530086090966721"/>
+            <inertia ixx="1.88176298336665E-05" ixy="-4.8444933029987E-10" ixz="1.88163708851143E-08"
+                    iyy="3.11510738647764E-05" iyz="-6.93560663069607E-11"
+                    izz="1.8801969558182E-05"/>
+        </inertial>
         <visual>
             <origin rpy="0 0 0" xyz="0 0 0"/>
@@ -9,4 +17,10 @@
             </geometry>
         </visual>
+        <collision>
+            <origin rpy="0 0 0" xyz="0 0 0"/>
+            <geometry>
+                <mesh filename="package://bumperbot_description/meshes/base_link.STL"/>
+            </geometry>
+        </collision>
     </link>
     <joint name="base_joint" type="fixed">
@@ -16,4 +30,11 @@
     </joint>
     <link name="wheel_right_link">
+        <inertial>
+            <origin xyz="0 0.014 0" rpy="0 0 0"/>
+            <mass value="0.0530086043217644"/>
+            <inertia ixx="1.8792911368909E-05" ixy="3.31256392204584E-10" ixz="-1.14082001662767E-08"
+                    iyy="3.11510738759073E-05" iyz="-3.60499245082192E-10"
+                    izz="1.88266886146847E-05"/>
+</inertial>
         <visual>
             <origin rpy="1.57 0 0" xyz="0 0 0"/>
@@ -22,4 +43,10 @@
             </geometry>
         </visual>
+        <collision>
+            <origin xyz="0 -.015 0" rpy="1.57 0 0" />
+            <geometry>
+                <sphere radius="0.033"/>
+            </geometry>
+        </collision>
     </link>
     <joint name="wheel_right_joint" type="continuous">
@@ -30,4 +57,11 @@
     </joint>
     <link name="wheel_left_link">
+        <inertial>
+            <origin xyz="0 0.014 0" rpy="0 0 0"/>
+            <mass value="0.0530086043217644"/>
+            <inertia ixx="1.8792911368909E-05" ixy="3.31256392204584E-10" ixz="-1.14082001662767E-08"
+                    iyy="3.11510738759073E-05" iyz="-3.60499245082192E-10"
+                    izz="1.88266886146847E-05"/>
+        </inertial>
         <visual>
             <origin rpy="-1.57 0 0" xyz="0 0 0"/>
@@ -36,4 +70,10 @@
             </geometry>
         </visual>
+        <collision>
+            <origin xyz="0 .015 0" rpy="1.57 0 0" />
+            <geometry>
+                <sphere radius="0.033"/>
+            </geometry>
+        </collision>
     </link>
     <joint name="wheel_left_joint" type="continuous">
@@ -44,4 +84,11 @@
     </joint>
     <link name="caster_front_link">
+        <inertial>
+            <origin xyz="3.89968128948481E-07 2.40073004698083E-07 0.00219173397061506" rpy="0 0 0"/>
+            <mass value="1.44379265037903E-06"/>
+            <inertia ixx="7.23075276010246E-11" ixy="-6.10956883467859E-16" ixz="2.22849693525031E-15"
+                    iyy="3.8713793085917E-11" iyz="2.93909858781952E-15"
+                    izz="1.00967486676306E-10"/>
+        </inertial>
         <visual>
             <origin rpy="0 0 0" xyz="0 0 0"/>
@@ -50,4 +97,10 @@
             </geometry>
         </visual>
+        <collision>
+            <origin rpy="0 0 0" xyz="0 0 0"/>
+            <geometry>
+                <sphere radius="0.005"/>
+            </geometry>
+        </collision>
     </link>
     <joint name="caster_front_joint" type="fixed">
@@ -57,4 +110,11 @@
     </joint>
     <link name="caster_rear_link">
+        <inertial>
+            <origin xyz="3.8996812895542E-07 2.40073004698083E-07 0.00219173397061509" rpy="0 0 0"/>
+            <mass value="1.44379265037902E-06"/>
+            <inertia ixx="7.23075276010246E-11" ixy="-6.10956872363424E-16" ixz="2.22849693527207E-15"
+                    iyy="3.87137930859167E-11" iyz="2.939098587861E-15"
+                    izz="1.00967486676306E-10"/>
+        </inertial>
         <visual>
             <origin rpy="0 0 0" xyz="0 0 0"/>
@@ -63,4 +123,10 @@
             </geometry>
         </visual>
+        <collision>
+            <origin rpy="0 0 0" xyz="0 0 0"/>
+            <geometry>
+                <sphere radius="0.005"/>
+            </geometry>
+        </collision>
     </link>
     <joint name="caster_rear_joint" type="fixed">
